File: readerIC.kicad_sch (KiCad schematic)
At the start: 62 parts, among them Q1 NPN, U1 BQ76952PFBR

Commit message: lots of lots changes. Schematic done NEEDS Review
Parts:
- added R47, R48: 0R, symbol Device:R
Connections:
- net GND: no longer R25.1, R26.1
- net at C13.2, C14.1, R14.2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: now also R48.1
- net at C14.2, C15.1, R15.2: now also R47.1; no longer R19.1, U1.2 (VC14)
- net at C26.1, U1.35 (REG1): no longer R28.2, R29.1
- new net: R19.1, R47.2, R48.2, U1.2 (VC14)
- new net +3V3: R28.2, R29.1
- new net GNDPWR: R25.1, R26.1
Other:
- note added: "Not: R18 ve R19 dirençler 14S için eğer 15s ya da 16S yapılacaksa R18, R19 ve R21 numaralı dirençler sökülmeli eğer 13s olacaksa R47 R21 Sökülmeli,"
- note removed: "Not: R18 ve R19 dirençler 14S için eğer 15s ya da 16S yapılacaksa R18 ve R19 dirençler sökülmeli R20 her türlü Takılmalı"
- company: (none) -> Pehlivan Team
- title: (none) -> BMS IC
Changed lines of the file:
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@@
 	(generator_version "9.0")
 	(paper "A4")
-	(text "Not:\nR18 ve R19 dirençler 14S için\neğer 15s ya da 16S yapılacaksa R18 ve R19 dirençler sökülmeli\nR20 her türlü Takılmalı\n"
+	(title_block
+		(title "BMS IC")
+		(date "2026-01-01")
+		(rev "0.1")
+		(company "Pehlivan Team")
+	)
+	(text "Not:\nR18 ve R19 dirençler 14S için\neğer 15s ya da 16S yapılacaksa R18, R19 ve R21 numaralı dirençler sökülmeli\neğer 13s olacaksa R47 R21 Sökülmeli,\n"
 		(exclude_from_sim no)
-		(at 132.08 174.752 0)
+		(at 135.382 172.974 0)
 		(effects
 			(font
@@
 	)
 	(junction
-		(at 227.33 54.61)
+		(at 148.59 59.69)
 		(diameter 0)
 		(color 0 0 0 0)
 	)
 	(junction
-		(at 148.59 59.69)
+		(at 130.81 132.08)
 		(diameter 0)
 		(color 0 0 0 0)
@@
 	)
 	(junction
-		(at 240.03 90.17)
-		(diameter 0)
-		(color 255 1 18 1)
-	)
-	(junction
 		(at 220.98 35.56)
 		(diameter 0)
@@
 	(wire
 		(pts
-			(xy 240.03 90.17) (xy 219.71 90.17)
-		)
-		(stroke
-			(width 0)
-			(type default)
-			(color 255 0 9 1)
-		)
-	)
-	(wire
-		(pts
 			(xy 167.64 151.13) (xy 171.45 151.13)
 		)
@@
 	(wire
 		(pts
-			(xy 240.03 107.95) (xy 219.71 107.95)
+			(xy 134.62 100.33) (xy 152.4 100.33)
 		)
 		(stroke
 			(width 0)
 			(type default)
-			(color 255 0 9 1)
 		)
 	)
 	(wire
 		(pts
-			(xy 134.62 100.33) (xy 152.4 100.33)
+			(xy 130.81 132.08) (xy 115.57 132.08)
 		)
 		(stroke
@@
 	(wire
 		(pts
-			(xy 138.43 132.08) (xy 115.57 132.08)
+			(xy 138.43 132.08) (xy 130.81 132.08)
 		)
 		(stroke
@@
 	(wire
 		(pts
-			(xy 240.03 54.61) (xy 240.03 90.17)
-		)
-		(stroke
-			(width 0)
-			(type default)
-			(color 255 0 9 1)
-		)
-	)
-	(wire
-		(pts
 			(xy 198.12 62.23) (xy 204.47 62.23)
 		)
@@
 	(wire
 		(pts
-			(xy 115.57 139.7) (xy 130.81 139.7)
+			(xy 115.57 139.7) (xy 123.19 139.7)
 		)
 		(stroke
@@
 	(wire
 		(pts
-			(xy 227.33 54.61) (xy 240.03 54.61)
-		)
-		(stroke
-			(width 0)
-			(type default)
-			(color 255 0 9 1)
-		)
-	)
-	(wire
-		(pts
 			(xy 95.25 19.05) (xy 165.1 19.05)
 		)
@@
 	(wire
 		(pts
+			(xy 223.52 90.17) (xy 219.71 90.17)
+		)
+		(stroke
+			(width 0)
+			(type default)
+		)
+	)
+	(wire
+		(pts
 			(xy 93.98 154.94) (xy 96.52 154.94)
 		)
@@
 	(wire
 		(pts
+			(xy 223.52 107.95) (xy 219.71 107.95)
+		)
+		(stroke
+			(width 0)
+			(type default)
+		)
+	)
+	(wire
+		(pts
 			(xy 139.7 82.55) (xy 152.4 82.55)
 		)
@@
 		)
 	)
-	(wire
-		(pts
-			(xy 240.03 90.17) (xy 240.03 107.95)
-		)
-		(stroke
-			(width 0)
-			(type default)
-			(color 255 0 9 1)
-		)
-	)
 	(global_label "BAT"
 		(shape input)
@@
 		)
 	)
+	(hierarchical_label "+3V3"
+		(shape input)
+		(at 223.52 107.95 0)
+		(effects
+			(font
+				(size 1.27 1.27)
+			)
+			(justify left)
+		)
+	)
 	(hierarchical_label "CI_Top"
 		(shape output)
@@
 		)
 	)
+	(hierarchical_label "+3V3"
+		(shape input)
+		(at 223.52 90.17 0)
+		(effects
+			(font
+				(size 1.27 1.27)
+			)
+			(justify left)
+		)
+	)
 	(symbol
 		(lib_id "Device:C")
@@
 	)
 	(symbol
+		(lib_id "power:GNDPWR")
+		(at 156.21 26.67 0)
+		(unit 1)
+		(exclude_from_sim no)
+		(in_bom yes)
+		(on_board yes)
+		(dnp no)
+		(fields_autoplaced yes)
+		(property "Reference" "#PWR08"
+			(at 156.21 31.75 0)
+			(effects
+				(font
+					(size 1.27 1.27)
+				)
+				(hide yes)
+			)
+		)
+		(property "Value" "GNDPWR"
+			(at 156.083 30.48 0)
+			(effects
+				(font
+					(size 1.27 1.27)
+				)
+			)
+		)
+		(property "Footprint" ""
+			(at 156.21 27.94 0)
+			(effects
+				(font
+					(size 1.27 1.27)
+				)
+				(hide yes)
+			)
+		)
+		(property "Datasheet" ""
+			(at 156.21 27.94 0)
+			(effects
+				(font
+					(size 1.27 1.27)
+				)
+				(hide yes)
+			)
+		)
+		(property "Description" "Power symbol creates a global label with name \"GNDPWR\" , global ground"
+			(at 156.21 26.67 0)
+			(effects
+				(font
+					(size 1.27 1.27)
+				)
+				(hide yes)
+			)
+		)
+		(pin "1"
+		)
+		(instances
+			(project "shell-bms"
+				(path "/ad9edf65-9f41-4da5-ac8d-b0754357a532/f6c14c9f-be18-4932-99a8-c7d510021503"
+					(reference "#PWR08")
+					(unit 1)
+				)
+			)
+		)
+	)
+	(symbol
 		(lib_id "Device:C")
 		(at 115.57 143.51 0)
@@
 	(symbol
 		(lib_id "Device:R")
+		(at 130.81 135.89 0)
+		(unit 1)
+		(exclude_from_sim no)
+		(in_bom yes)
+		(on_board yes)
+		(dnp no)
+		(property "Reference" "R48"
+			(at 132.334 135.89 0)
+			(effects
+				(font
+					(size 1.27 1.27)
+				)
+				(justify left)
+			)
+		)
+		(property "Value" "0R"
+			(at 131.064 136.906 90)
+			(effects
+				(font
+					(size 1.27 1.27)
+				)
+				(justify left)
+			)
+		)
+		(property "Footprint" ""
+			(at 129.032 135.89 90)
+			(effects
+				(font
+					(size 1.27 1.27)
+				)
+				(hide yes)
+			)
+		)
+		(property "Datasheet" "~"
+			(at 130.81 135.89 0)
+			(effects
+				(font
+					(size 1.27 1.27)
+				)
+				(hide yes)
+			)
+		)
+		(property "Description" "Resistor"
+			(at 130.81 135.89 0)
+			(effects
+				(font
+					(size 1.27 1.27)
+				)
+				(hide yes)
+			)
+		)
+		(pin "1"
+		)
+		(pin "2"
+		)
+		(instances
+			(project "shell-bms"
+				(path "/ad9edf65-9f41-4da5-ac8d-b0754357a532/f6c14c9f-be18-4932-99a8-c7d510021503"
+					(reference "R48")
+					(unit 1)
+				)
+			)
+		)
+	)
+	(symbol
+		(lib_id "Device:R")
 		(at 219.71 104.14 0)
 		(unit 1)
@@
 	(symbol
 		(lib_id "power:GND")
-		(at 156.21 26.67 0)
+		(at 22.86 140.97 270)
 		(unit 1)
 		(exclude_from_sim no)
@@
 		(dnp no)
 		(fields_autoplaced yes)
-		(property "Reference" "#PWR08"
-			(at 156.21 33.02 0)
+		(property "Reference" "#PWR05"
+			(at 16.51 140.97 0)
 			(effects
 				(font
@@
 		)
 		(property "Value" "GND"
-			(at 156.21 31.75 0)
+			(at 19.05 140.9699 90)
 			(effects
 				(font
 					(size 1.27 1.27)
 				)
+				(justify right)
 			)
 		)
 		(property "Footprint" ""
-			(at 156.21 26.67 0)
+			(at 22.86 140.97 0)
 			(effects
 				(font
@@
 		)
 		(property "Datasheet" ""
-			(at 156.21 26.67 0)
+			(at 22.86 140.97 0)
 			(effects
 				(font
@@
 		)
 		(property "Description" "Power symbol creates a global label with name \"GND\" , ground"
-			(at 156.21 26.67 0)
+			(at 22.86 140.97 0)
 			(effects
 				(font
@@
 			(project ""
 				(path "/ad9edf65-9f41-4da5-ac8d-b0754357a532/f6c14c9f-be18-4932-99a8-c7d510021503"
-					(reference "#PWR08")
+					(reference "#PWR05")
 					(unit 1)
 				)
@@
 	)
 	(symbol
-		(lib_id "power:GND")
-		(at 22.86 140.97 270)
+		(lib_id "Device:R")
+		(at 127 139.7 90)
 		(unit 1)
 		(exclude_from_sim no)
@@
 		(on_board yes)
 		(dnp no)
-		(fields_autoplaced yes)
-		(property "Reference" "#PWR05"
-			(at 16.51 140.97 0)
+		(property "Reference" "R47"
+			(at 127 141.986 90)
 			(effects
 				(font
 					(size 1.27 1.27)
 				)
-				(hide yes)
 			)
 		)
-		(property "Value" "GND"
-			(at 19.05 140.9699 90)
+		(property "Value" "0R"
+			(at 127 139.7 90)
 			(effects
 				(font
 					(size 1.27 1.27)
 				)
-				(justify right)
 			)
 		)
 		(property "Footprint" ""
-			(at 22.86 140.97 0)
+			(at 127 141.478 90)
 			(effects
 				(font
@@
 			)
 		)
-		(property "Datasheet" ""
-			(at 22.86 140.97 0)
+		(property "Datasheet" "~"
+			(at 127 139.7 0)
 			(effects
 				(font
@@
 			)
 		)
-		(property "Description" "Power symbol creates a global label with name \"GND\" , ground"
-			(at 22.86 140.97 0)
+		(property "Description" "Resistor"
+			(at 127 139.7 0)
 			(effects
 				(font
@@
 		(pin "1"
 		)
+		(pin "2"
+		)
 		(instances
-			(project ""
+			(project "shell-bms"
 				(path "/ad9edf65-9f41-4da5-ac8d-b0754357a532/f6c14c9f-be18-4932-99a8-c7d510021503"
-					(reference "#PWR05")
+					(reference "R47")
 					(unit 1)
 				)

Commit message: son update
Parts:
- added R61: 1m, Resistor_SMD:R_0603_1608Metric_Pad0.98x0.95mm_HandSolder, symbol Device:R
- C1, C10, C11, C12, C13, C14, C15, C16, C17, C18, C19, C2, C20, C3, C4, C5, C6, C7, C8, C9: footprint (none) -> Capacitor_SMD:C_1210_3225Metric_Pad1.33x2.70mm_HandSolder
- C21, C22, C23, C24, C25, C26, C27, C28: footprint (none) -> Capacitor_SMD:C_0805_2012Metric_Pad1.18x1.45mm_HandSolder
- D1: footprint (none) -> Diode_THT:D_A-405_P7.62mm_Horizontal
- Q1: footprint (none) -> Package_TO_SOT_THT:TO-92_HandSolder
- R1, R10, R11, R12, R13, R14, R15, R16, R17, R18, R19, R2, R20, R21, R3, R4, R5, R6, R7, R8, R9: footprint (none) -> Resistor_SMD:R_1210_3225Metric_Pad1.30x2.65mm_HandSolder
- R22, R23, R24, R25, R26, R27, R28, R29, R30: footprint (none) -> Resistor_THT:R_Axial_DIN0309_L9.0mm_D3.2mm_P15.24mm_Horizontal
- R47, R48: footprint (none) -> Resistor_SMD:R_0603_1608Metric_Pad0.98x0.95mm_HandSolder
- U1: footprint BQ76952PFBR:QFP50P900X900X120-48N -> BQ76952:QFP50P900X900X120-48N
Connections:
- net Balance-Input/B_0: now also R61.2
- net GNDPWR: now also R61.1
- net CI_Top renamed Balance-Input/B_16
- no-connect marks 3 -> 6
