File: readerIC.kicad_sch (KiCad schematic)
At the start: 65 parts, among them Q1 NPN, U1 BQ76952PFBR

Commit message: bit artık
Parts:
- R23, R24, R28, R29: footprint Resistor_THT:R_Axial_DIN0309_L9.0mm_D3.2mm_P15.24mm_Horizontal -> Resistor_SMD:R_1210_3225Metric_Pad1.30x2.65mm_HandSolder
Connections:
- net Balance-Input/B_0: no longer C1.2, R1.2, U1.16 (VC0)
- net GND: no longer C21.1, C22.1, C27.1
- net GNDPWR: now also C21.1, C22.1, C27.1; no longer C17.1
- new net: C1.2, C17.1, R1.2, U1.16 (VC0)
Other:
- moved on the sheet: C1

Commit message: BMS DONE IHOPE
Parts:
- removed R25: 1m, Resistor_SMD:R_1210_3225Metric_Pad1.30x2.65mm_HandSolder, symbol Device:R
- C1, C10, C11, C12, C13, C14, C15, C16, C17, C2, C3, C4, C5, C6, C7, C8, C9: footprint Capacitor_SMD:C_1210_3225Metric_Pad1.33x2.70mm_HandSolder -> Capacitor_SMD:C_0805_2012Metric_Pad1.18x1.45mm_HandSolder
- R23, R24, R26, R27, R28, R29: footprint Resistor_SMD:R_1210_3225Metric_Pad1.30x2.65mm_HandSolder -> Resistor_SMD:R_0603_1608Metric_Pad0.98x0.95mm_HandSolder
- R30: value R -> 300; footprint Resistor_THT:R_Axial_DIN0309_L9.0mm_D3.2mm_P15.24mm_Horizontal -> Resistor_SMD:R_0805_2012Metric_Pad1.20x1.40mm_HandSolder
Connections:
- net +3V3: now also R28.1, R29.2; no longer R28.2, R29.1
- net GNDPWR: now also R27.1, R61.2
- net IC_SCL: now also R28.2; no longer R29.2
- net IC_SDA: now also R29.1; no longer R28.1
- removed net Balance-Input/B_0: R1.1, R27.1, R61.2
- net Balance-Input/B_1 renamed Balance-Input/CI_1
- net Balance-Input/B_10 renamed Balance-Input/CI_10
- net Balance-Input/B_11 renamed Balance-Input/CI_11
- net Balance-Input/B_12 renamed Balance-Input/CI_12
- net Balance-Input/B_13 renamed Balance-Input/CI_13
- net Balance-Input/B_14 renamed Balance-Input/CI_14
- net Balance-Input/B_15 renamed Balance-Input/CI_15
- net Balance-Input/B_16 renamed Balance-Input/CI_16
- net Balance-Input/B_2 renamed Balance-Input/CI_2
- net Balance-Input/B_3 renamed Balance-Input/CI_3
- net Balance-Input/B_4 renamed Balance-Input/CI_4
- net Balance-Input/B_5 renamed Balance-Input/CI_5
- net Balance-Input/B_6 renamed Balance-Input/CI_6
- net Balance-Input/B_7 renamed Balance-Input/CI_7
- net Balance-Input/B_8 renamed Balance-Input/CI_8
- net Balance-Input/B_9 renamed Balance-Input/CI_9
- new net Balance-Input/CI_0: R1.1
Other:
- sheet Balance-Input ports: added none; removed B_0, B_1, B_10, B_11, B_12, B_13, B_14, B_15, B_16, B_2, B_3, B_4, B_5, B_6, B_7, B_8, B_9, GND
- note added: "Not: R18 ve R19 dirençler 14S için eğer 15s ya da 16S yapılacaksa R18, R19 ve R21 numaralı dirençler sökülmeli eğer 13s olacaksa R47 R21 Sökülmeli,sökülmeli"
- note removed: "Not: R18 ve R19 dirençler 14S için eğer 15s ya da 16S yapılacaksa R18, R19 ve R21 numaralı dirençler sökülmeli eğer 13s olacaksa R47 R21 Sökülmeli,"
- moved on the sheet: R28, R29
