File: balancer.kicad_sch (KiCad schematic)
At the start: 3 parts, among them J1 Conn_01x20, J2 Conn_01x20, J3 Conn_01x04

Commit message: lots of lots changes. Schematic done NEEDS Review
Other:
- company: (none) -> Pehlivan Team
- title: (none) -> Balance And Balance Cable Input
- moved on the sheet: J3
Changed lines of the file:
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@@
 	(generator_version "9.0")
 	(paper "A4")
+	(title_block
+		(title "Balance And Balance Cable Input")
+		(date "2026-01-01")
+		(rev "0.1")
+		(company "Pehlivan Team")
+	)
 	(no_connect
 		(at 113.03 113.03)
@@
 	(hierarchical_label "TS2"
 		(shape input)
-		(at 113.03 125.73 180)
+		(at 137.16 132.08 270)
 		(effects
 			(font
@@
 	(hierarchical_label "GND"
 		(shape input)
-		(at 113.03 130.81 180)
+		(at 142.24 132.08 270)
 		(effects
 			(font
@@
 	(hierarchical_label "TS1"
 		(shape input)
-		(at 113.03 123.19 180)
+		(at 134.62 132.08 270)
 		(effects
 			(font
@@
 	(hierarchical_label "TS3"
 		(shape input)
-		(at 113.03 128.27 180)
+		(at 139.7 132.08 270)
 		(effects
 			(font
@@
 	(symbol
 		(lib_id "Connector_Generic:Conn_01x04")
-		(at 118.11 125.73 0)
+		(at 137.16 127 90)
 		(unit 1)
 		(exclude_from_sim no)
@@
 		(fields_autoplaced yes)
 		(property "Reference" "J3"
-			(at 120.65 125.7299 0)
+			(at 137.1599 124.46 0)
 			(effects
 				(font
@@
 		)
 		(property "Value" "Conn_01x04"
-			(at 120.65 128.2699 0)
+			(at 139.6999 124.46 0)
 			(effects
 				(font
@@
 		)
 		(property "Footprint" ""
-			(at 118.11 125.73 0)
+			(at 137.16 127 0)
 			(effects
 				(font
@@
 		)
 		(property "Datasheet" "~"
-			(at 118.11 125.73 0)
+			(at 137.16 127 0)
 			(effects
 				(font
@@
 		)
 		(property "Description" "Generic connector, single row, 01x04, script generated (kicad-library-utils/schlib/autogen/connector/)"
-			(at 118.11 125.73 0)
-			(effects
-				(font
+			(at 137.16 127 0)
+			(effects
+				(font

Commit message: son update
Parts:
- J1, J2: footprint (none) -> Connector_PinSocket_2.54mm:PinSocket_1x20_P2.54mm_Vertical_SMD_Pin1Right
- J3: footprint (none) -> Connector_PinSocket_2.54mm:PinSocket_1x04_P2.54mm_Vertical
Changed lines of the file:
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@@
 			)
 		)
-		(property "Footprint" ""
+		(property "Footprint" "Connector_PinSocket_2.54mm:PinSocket_1x20_P2.54mm_Vertical_SMD_Pin1Right"
 			(at 118.11 92.71 0)
 			(effects
@@
 			)
 		)
-		(property "Footprint" ""
+		(property "Footprint" "Connector_PinSocket_2.54mm:PinSocket_1x04_P2.54mm_Vertical"
 			(at 137.16 127 0)
 			(effects
@@
 			)
 		)
-		(property "Footprint" ""
+		(property "Footprint" "Connector_PinSocket_2.54mm:PinSocket_1x20_P2.54mm_Vertical_SMD_Pin1Right"
 			(at 165.1 92.71 0)
 			(effects

Commit message: bit artık
Parts:
- J2: footprint Connector_PinSocket_2.54mm:PinSocket_1x20_P2.54mm_Vertical_SMD_Pin1Right -> Connector_PinSocket_2.54mm:PinSocket_1x20_P2.54mm_Horizontal
Connections:
- net GND renamed GNDPWR
Changed lines of the file:
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@@
+	)
+	(no_connect
+		(at 160.02 113.03)
+	)
+	(no_connect
+		(at 113.03 115.57)
 	)
 	(no_connect
 		(at 113.03 118.11)
 	)
-	(no_connect
-		(at 160.02 113.03)
-	)
-	(no_connect
-		(at 113.03 115.57)
-	)
 	(hierarchical_label "CI_4"
 		(shape input)
@@
 		)
 	)
-	(hierarchical_label "GND"
-		(shape input)
-		(at 142.24 132.08 270)
+	(hierarchical_label "NTC+"
+		(shape input)
+		(at 160.02 115.57 180)
 		(effects
 			(font
@@
 		)
 	)
+	(hierarchical_label "NTC-"
+		(shape input)
+		(at 160.02 118.11 180)
+		(effects
+			(font
+				(size 1.27 1.27)
+			)
+			(justify right)
+		)
+	)
 	(hierarchical_label "B_5"
 		(shape input)
@@
 		)
 	)
-	(hierarchical_label "NTC+"
-		(shape input)
-		(at 160.02 115.57 180)
-		(effects
-			(font
-				(size 1.27 1.27)
-			)
-			(justify right)
-		)
-	)
 	(hierarchical_label "B_11"
 		(shape input)
@@
 		(shape input)
 		(at 160.02 105.41 180)
-		(effects
-			(font
-				(size 1.27 1.27)
-			)
-			(justify right)
-		)
-	)
-	(hierarchical_label "NTC-"
-		(shape input)
-		(at 160.02 118.11 180)
 		(effects
 			(font
@@
 			)
 		)
-		(property "Footprint" "Connector_PinSocket_2.54mm:PinSocket_1x20_P2.54mm_Vertical_SMD_Pin1Right"
+		(property "Footprint" "Connector_PinSocket_2.54mm:PinSocket_1x20_P2.54mm_Horizontal"
 			(at 118.11 92.71 0)
 			(effects
@@
 					(unit 1)
 				)
+			)
+		)
+	)
+	(symbol
+		(lib_id "power:GNDPWR")
+		(at 142.24 132.08 0)
+		(unit 1)
+		(exclude_from_sim no)
+		(in_bom yes)
+		(on_board yes)
+		(dnp no)
+		(fields_autoplaced yes)
+		(property "Reference" "#PWR063"
+			(at 142.24 137.16 0)
+			(effects
+				(font
+					(size 1.27 1.27)
+				)
+				(hide yes)
+			)
+		)
+		(property "Value" "GNDPWR"
+			(at 142.113 135.89 0)
+			(effects
+				(font
+					(size 1.27 1.27)
+				)
+			)
+		)
+		(property "Footprint" ""
+			(at 142.24 133.35 0)
+			(effects
+				(font
+					(size 1.27 1.27)
+				)
+				(hide yes)
+			)
+		)
+		(property "Datasheet" ""
+			(at 142.24 133.35 0)
+			(effects
+				(font
+					(size 1.27 1.27)
+				)
+				(hide yes)
+			)
+		)
+		(property "Description" "Power symbol creates a global label with name \"GNDPWR\" , global ground"
+			(at 142.24 132.08 0)
+			(effects
+				(font
+					(size 1.27 1.27)
+				)
+				(hide yes)
+			)
+		)
+		(pin "1"
+		)
+		(instances
+			(project ""
+				(path "/ad9edf65-9f41-4da5-ac8d-b0754357a532/f6c14c9f-be18-4932-99a8-c7d510021503/e7e6bd43-5535-45bf-89a8-507685ee23ac"
+					(reference "#PWR063")
+					(unit 1)
+				)

Commit message: BMS DONE IHOPE
Parts:
- removed J1: Conn_01x20, Connector_PinSocket_2.54mm:PinSocket_1x20_P2.54mm_Vertical_SMD_Pin1Right, symbol Connector_Generic:Conn_01x20
- J2: footprint Connector_PinSocket_2.54mm:PinSocket_1x20_P2.54mm_Horizontal -> Connector_Wago:Wago_734-180_1x20_P3.50mm_Horizontal
Connections:
- net CI_0: now also J2.17 (Pin_17); no longer J2.1 (Pin_1)
- net CI_1: now also J2.16 (Pin_16); no longer J2.2 (Pin_2)
- net CI_10: now also J2.7 (Pin_7); no longer J2.11 (Pin_11)
- net CI_11: now also J2.6 (Pin_6); no longer J2.12 (Pin_12)
- net CI_12: now also J2.5 (Pin_5); no longer J2.13 (Pin_13)
- net CI_13: now also J2.4 (Pin_4); no longer J2.14 (Pin_14)
- net CI_14: now also J2.3 (Pin_3); no longer J2.15 (Pin_15)
- net CI_15: now also J2.2 (Pin_2); no longer J2.16 (Pin_16)
- net CI_16: now also J2.1 (Pin_1); no longer J2.17 (Pin_17)
- net CI_2: now also J2.15 (Pin_15); no longer J2.3 (Pin_3)
- net CI_3: now also J2.14 (Pin_14); no longer J2.4 (Pin_4)
- net CI_4: now also J2.13 (Pin_13); no longer J2.5 (Pin_5)
- net CI_5: now also J2.12 (Pin_12); no longer J2.6 (Pin_6)
- net CI_6: now also J2.11 (Pin_11); no longer J2.7 (Pin_7)
- net CI_7: now also J2.10 (Pin_10); no longer J2.8 (Pin_8)
- net CI_9: now also J2.8 (Pin_8); no longer J2.10 (Pin_10)
- net NTC+: now also J2.19 (Pin_19)
- net NTC-: now also J2.20 (Pin_20)
- no-connect marks 4 -> 1
Other:
- moved on the sheet: J3
