File: mcu.kicad_sch (KiCad schematic)
At the start: 1 part, among them U3 STM32G431C8Tx

Commit message: lots of lots changes. Schematic done NEEDS Review
Parts:
- added C42, C43, C44, C47 (x2), C48, C50, C52, C54: 100nF, Capacitor_SMD:C_0603_1608Metric_Pad1.08x0.95mm_HandSolder, symbol Device:C
- added C45, C46 (x2), C53: 10uF, Capacitor_SMD:C_0603_1608Metric_Pad1.08x0.95mm_HandSolder, symbol Device:C
- added C49: 1uF, Capacitor_SMD:C_0603_1608Metric_Pad1.08x0.95mm_HandSolder, symbol Device:C
- added C51: 10uf, Capacitor_SMD:C_0805_2012Metric_Pad1.18x1.45mm_HandSolder, symbol Device:C
- added C56, C57: 22pF, Capacitor_SMD:C_0603_1608Metric_Pad1.08x0.95mm_HandSolder, symbol Device:C
- added C58: 100nF, Capacitor_THT:C_Disc_D10.5mm_W5.0mm_P5.00mm, symbol Device:C
- added FB1: 12R, Resistor_SMD:R_0805_2012Metric_Pad1.20x1.40mm_HandSolder, symbol Device:FerriteBead
- added J9: Conn_01x04, symbol Connector_Generic:Conn_01x04
- added R55: 10K, Resistor_THT:R_Axial_DIN0207_L6.3mm_D2.5mm_P7.62mm_Horizontal, symbol Device:R
- added SW1: SW_Push, Button_Switch_THT:SW_PUSH_6mm_H8mm, symbol Switch:SW_Push
- added Y1: 8MHz, Crystal:Crystal_HC18-U_Vertical, symbol Device:Crystal
Connections:
- net GND: now also C42.1, C43.1, C44.1, C45.1, C46.1, C46.1, C47.1, C47.1, C48.1, C49.2, C50.2, C51.2, C52.1, C53.1, C54.1, C56.1, C57.1, C58.1, J9.4 (Pin_4), SW1.1
- net +3V3: now reaches U3.1 (VBAT)
- net +3V3: now also U3.24 (VDD), U3.36 (VDD), U3.48 (VDD), C42.2, C43.2, C44.2, C45.2, C46.2, C46.2, C47.2, C47.2, C48.2, C51.1, C52.2, C53.2, C54.2, FB1.2, J9.3 (Pin_3), R55.2
- net UART_USB_TX: now reaches U3.10 (PA2)
- net UART_USB_RX: now reaches U3.11 (PA3)
- net VREF+: now reaches U3.20 (VREF+)
- net VREF+: now also U3.21 (VDDA), C49.1, C50.1, FB1.1
- net BUZZER: now reaches U3.27 (PB13)
- net STAT_LED: now reaches U3.28 (PB14)
- net IC_SDA: now reaches U3.30 (PA8)
- net IC_SCL: now reaches U3.31 (PA9)
- net CAN_RX: now reaches U3.33 (PA11)
- net CAN_TX: now reaches U3.34 (PA12)
- net at U3.37 (PA13): now also J9.1 (Pin_1)
- net at U3.38 (PA14): now also J9.2 (Pin_2)
- net PB3: now reaches U3.40 (PB3)
- net PB4: now reaches U3.41 (PB4)
- net PB5: now reaches U3.42 (PB5)
- net at U3.5 (PF0): now also C56.2, Y1.1
- net at U3.6 (PF1): now also C57.2, Y1.2
- net NRST: now reaches U3.7 (PG10)
- net NRST: now also C58.2, R55.1, SW1.2
- net FAN2: now reaches U3.8 (PA0)
- net FAN1: now reaches U3.9 (PA1)
- no-connect marks 0 -> 19
Other:
- company: (none) -> Pehlivan Team
- title: (none) -> MCU
- moved on the sheet: U3

Commit message: son update
Parts:
- J9: footprint (none) -> Connector_PinSocket_2.00mm:PinSocket_1x04_P2.00mm_Vertical
- renumbered C46 to C59, C47 to C60
Connections:
- net NTC: now reaches U3.12 (PA4)
Other:
- added sheet esp32 (esp.kicad_sch)
Changed lines of the file:
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@@
 	)
 	(no_connect
-		(at 177.8 96.52)
-	)
-	(no_connect
 		(at 177.8 104.14)
 	)
@@
 	)
 	(no_connect
+		(at 142.24 152.4)
+	)
+	(no_connect
 		(at 142.24 114.3)
 	)
@@
 		)
 	)
+	(hierarchical_label "NTC"
+		(shape input)
+		(at 177.8 96.52 0)
+		(effects
+			(font
+				(size 1.27 1.27)
+			)
+			(justify left)
+		)
+	)
 	(hierarchical_label "UART_USB_RX"
 		(shape output)
@@
 		(on_board yes)
 		(dnp no)
-		(fields_autoplaced yes)
-		(property "Reference" "C46"
-			(at 140.9701 45.72 0)
+		(property "Reference" "C59"
+			(at 142.24 44.196 0)
 			(effects
 				(font
 					(size 1.27 1.27)
 				)
-				(justify left)
 			)
 		)
 		(property "Value" "10uF"
-			(at 138.4301 45.72 0)
+			(at 137.668 44.196 0)
 			(effects
 				(font
 					(size 1.27 1.27)
 				)
-				(justify left)
 			)
 		)
@@
 			(project "shell-bms"
 				(path "/ad9edf65-9f41-4da5-ac8d-b0754357a532/539ae960-93b7-4680-b2d3-38d1676c29f9"
-					(reference "C46")
+					(reference "C59")
 					(unit 1)
 				)
@@
 			)
 		)
-		(property "Footprint" ""
+		(property "Footprint" "Connector_PinSocket_2.00mm:PinSocket_1x04_P2.00mm_Vertical"
 			(at 195.58 121.92 0)
 			(effects
@@
 		(on_board yes)
 		(dnp no)
-		(fields_autoplaced yes)
-		(property "Reference" "C47"
-			(at 140.9701 59.69 0)
+		(property "Reference" "C60"
+			(at 141.986 60.198 0)
 			(effects
 				(font
 					(size 1.27 1.27)
 				)
-				(justify left)
 			)
 		)
 		(property "Value" "100nF"
-			(at 138.4301 59.69 0)
+			(at 137.414 59.69 0)
 			(effects
 				(font
 					(size 1.27 1.27)
 				)
-				(justify left)
 			)
 		)
@@
 			(project "shell-bms"
 				(path "/ad9edf65-9f41-4da5-ac8d-b0754357a532/539ae960-93b7-4680-b2d3-38d1676c29f9"
-					(reference "C47")
+					(reference "C60")
 					(unit 1)
 				)
@@
 				)
 			)
+		)
+	)
+	(sheet
+		(at 41.91 147.32)
+		(size 29.21 20.32)
+		(exclude_from_sim no)
+		(in_bom yes)
+		(on_board yes)
+		(dnp no)
+		(fields_autoplaced yes)
+		(stroke
+			(width 0.1524)
+			(type solid)
+		)
+		(fill
+			(color 0 0 0 0.0000)
+		)
+		(property "Sheetname" "esp32"
+			(at 41.91 146.6084 0)
+			(effects
+				(font
+					(size 1.27 1.27)
+				)
+				(justify left bottom)
+			)
+		)
+		(property "Sheetfile" "esp.kicad_sch"
+			(at 41.91 168.2246 0)
+			(effects
+				(font
+					(size 1.27 1.27)
+				)
+				(justify left top)
+			)
+		)
+		(instances
+			(project "shell-bms"
+				(path "/ad9edf65-9f41-4da5-ac8d-b0754357a532/539ae960-93b7-4680-b2d3-38d1676c29f9"
+					(page "9")
+				)
+			)

Commit message: finalised product
Other:
- sheet esp32 ports: added 3V3, ESP_RX, ESP_TX; removed none
Changed lines of the file:
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@@
 		(color 0 0 0 0)
 	)
+	(junction
+		(at 203.2 92.71)
+		(diameter 0)
+		(color 0 0 0 0)
+	)
+	(junction
+		(at 200.66 93.98)
+		(diameter 0)
+		(color 0 0 0 0)
+	)
 	(no_connect
 		(at 142.24 132.08)
@@
 	(wire
 		(pts
-			(xy 177.8 93.98) (xy 198.12 93.98)
+			(xy 177.8 93.98) (xy 200.66 93.98)
 		)
 		(stroke
@@
 	(wire
 		(pts
+			(xy 214.63 96.52) (xy 217.17 96.52)
+		)
+		(stroke
+			(width 0)
+			(type default)
+		)
+	)
+	(wire
+		(pts
+			(xy 217.17 92.71) (xy 203.2 92.71)
+		)
+		(stroke
+			(width 0)
+			(type default)
+		)
+	)
+	(wire
+		(pts
+			(xy 203.2 92.71) (xy 199.39 92.71)
+		)
+		(stroke
+			(width 0)
+			(type default)
+		)
+	)
+	(wire
+		(pts
 			(xy 143.51 24.13) (xy 143.51 27.94)
 		)
@@
 	(wire
 		(pts
-			(xy 177.8 91.44) (xy 198.12 91.44)
+			(xy 177.8 91.44) (xy 199.39 91.44)
 		)
 		(stroke
@@
 	(wire
 		(pts
+			(xy 199.39 92.71) (xy 199.39 91.44)
+		)
+		(stroke
+			(width 0)
+			(type default)
+		)
+	)
+	(wire
+		(pts
 			(xy 157.48 78.74) (xy 157.48 72.39)
 		)
@@
 	(wire
 		(pts
+			(xy 200.66 93.98) (xy 214.63 93.98)
+		)
+		(stroke
+			(width 0)
+			(type default)
+		)
+	)
+	(wire
+		(pts
 			(xy 182.88 116.84) (xy 177.8 116.84)
 		)
@@
 	(wire
 		(pts
+			(xy 200.66 93.98) (xy 200.66 95.25)
+		)
+		(stroke
+			(width 0)
+			(type default)
+		)
+	)
+	(wire
+		(pts
 			(xy 124.46 27.94) (xy 124.46 41.91)
 		)
@@
 	(wire
 		(pts
+			(xy 203.2 92.71) (xy 203.2 95.25)
+		)
+		(stroke
+			(width 0)
+			(type default)
+		)
+	)
+	(wire
+		(pts
 			(xy 172.72 72.39) (xy 184.15 72.39)
 		)
@@
 	(wire
 		(pts
+			(xy 214.63 93.98) (xy 214.63 96.52)
+		)
+		(stroke
+			(width 0)
+			(type default)
+		)
+	)
+	(wire
+		(pts
 			(xy 154.94 27.94) (xy 154.94 41.91)
 		)
@@
 	(hierarchical_label "UART_USB_TX"
 		(shape output)
-		(at 198.12 91.44 0)
+		(at 203.2 95.25 270)
 		(effects
 			(font
 				(size 1.27 1.27)
 			)
-			(justify left)
+			(justify right)
 		)
 	)
@@
 	(hierarchical_label "UART_USB_RX"
 		(shape output)
-		(at 198.12 93.98 0)
+		(at 200.66 95.25 270)
 		(effects
 			(font
 				(size 1.27 1.27)
 			)
-			(justify left)
+			(justify right)
 		)
 	)
@@
 	)
 	(sheet
-		(at 41.91 147.32)
+		(at 217.17 85.09)
 		(size 29.21 20.32)
 		(exclude_from_sim no)
@@
 		)
 		(property "Sheetname" "esp32"
-			(at 41.91 146.6084 0)
+			(at 217.17 84.3784 0)
 			(effects
 				(font
@@
 		)
 		(property "Sheetfile" "esp.kicad_sch"
-			(at 41.91 168.2246 0)
+			(at 217.17 105.9946 0)
 			(effects
 				(font
@@
 			)
 		)
+		(pin "3V3" input
+			(at 219.71 85.09 90)
+			(effects
+				(font
+					(size 1.27 1.27)
+				)
+				(justify right)
+			)
+		)
+		(pin "ESP_TX" output
+			(at 217.17 92.71 180)
+			(effects
+				(font
+					(size 1.27 1.27)
+				)
+				(justify left)
+			)
+		)
+		(pin "ESP_RX" input
+			(at 217.17 96.52 180)
+			(effects
+				(font
+					(size 1.27 1.27)
+				)
+				(justify left)
+			)
+		)

Commit message: BMS DONE IHOPE
Parts:
- added J4: Conn_01x04, Connector_PinSocket_2.00mm:PinSocket_1x04_P2.00mm_Vertical, symbol Connector_Generic:Conn_01x04
Connections:
- net +3V3: now also J4.3 (Pin_3)
- net CAN_RX: now also U3.45 (PB8); no longer U3.33 (PA11)
- net CAN_TX: now also U3.46 (PB9); no longer U3.34 (PA12)
- net GND: now also J4.4 (Pin_4)
- net PB0: now reaches U3.16 (PB0)
- net PB1: now reaches U3.17 (PB1)
- net PB2: now reaches U3.18 (PB2)
- net I2C_SCL: now reaches U3.39 (PA15)
- net I2C_SCL: now also J4.1 (Pin_1)
- net PB6: now reaches U3.43 (PB6)
- net I2C_SDA: now reaches U3.44 (PB7)
- net I2C_SDA: now also J4.2 (Pin_2)
- net UART_USB_RX renamed esp32/ESP_RX
- net UART_USB_TX renamed esp32/ESP_TX
- new net USB+: U3.33 (PA11)
- new net USB-: U3.34 (PA12)
- no-connect marks 19 -> 11
Other:
- sheet esp32 ports: added none; removed 3V3
- moved on the sheet: J9
