File: protection.kicad_sch (KiCad schematic)
At the start: 25 parts, among them J4 Conn_01x04, Q2 NMOS, Q3 NMOS, Q4 NMOS

Commit message: lots of lots changes. Schematic done NEEDS Review
Parts:
- removed C31, C32: 0.1uF, symbol Device:C
- removed D5: 16V Zener, symbol Device:D_Zener
- removed D6, D7: 100V Zener, symbol Device:D_Zener
- removed Q4: NMOS, Package_TO_SOT_THT:TO-220-3_Vertical, symbol Simulation_SPICE:NMOS
- removed R40: 1M, symbol Device:R
- removed R41: 10K, symbol Device:R
- removed R42: 7.5K, symbol Device:R
- added R60: 2k, symbol Device:R
- J4: value Conn_01x04 -> Output
- Q2, Q3: value NMOS -> HY3610P
- R31: value R -> 2k
- R37, R38: value 5.1k -> 2k
Connections:
- net CHG: now also R60.2; no longer R31.2
- net CI_TOP renamed B_Pos
- net GND renamed GNDPWR
- new net: R31.2, R60.1
Other:
- company: (none) -> Pehlivan Team
- title: (none) -> Pehli-Shell-BMS
- moved on the sheet: C29, C30, D3, D4, Q2, Q3, R31, R32, R33, R34, R35, R36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

Commit message: son update
Parts:
- C29, C30: footprint (none) -> Capacitor_SMD:C_0805_2012Metric_Pad1.18x1.45mm_HandSolder
- D3, D4: footprint (none) -> Diode_THT:D_DO-201_P15.24mm_Horizontal
- J4: footprint (none) -> Connector_AMASS:AMASS_XT60-F_1x02_P7.20mm_Vertical; symbol Connector_Generic:Conn_01x04 -> Connector_Generic:Conn_01x02
- R31, R32, R37, R38, R39: footprint (none) -> Resistor_THT:R_Axial_DIN0309_L9.0mm_D3.2mm_P15.24mm_Horizontal
- R33, R34, R35, R36: footprint (none) -> Resistor_SMD:R_0508_1220Metric_Pad1.12x2.15mm_HandSolder
- R60: footprint (none) -> Resistor_SMD:R_0603_1608Metric_Pad0.98x0.95mm_HandSolder
Connections:
- net GNDPWR: now also J4.2 (Pin_2); no longer J4.3 (Pin_3), J4.4 (Pin_4)
- net at C30.2, D4.2 (A), J4.1 (Pin_1)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: no longer J4.2 (Pin_2)
Changed lines of the file:
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@@
-	)
-	(junction
-		(at 179.07 100.33)
-		(diameter 0)
-		(color 0 0 0 0)
 	)
 	(junction
@@
 	)
 	(junction
-		(at 179.07 93.98)
-		(diameter 0)
-		(color 0 0 0 0)
-	)
-	(junction
 		(at 68.58 93.98)
 		(diameter 0)
@@
 	(wire
 		(pts
-			(xy 179.07 93.98) (xy 181.61 93.98)
-		)
-		(stroke
-			(width 0)
-			(type default)
-		)
-	)
-	(wire
-		(pts
 			(xy 87.63 116.84) (xy 87.63 119.38)
 		)
@@
 	(wire
 		(pts
-			(xy 179.07 101.6) (xy 181.61 101.6)
-		)
-		(stroke
-			(width 0)
-			(type default)
-		)
-	)
-	(wire
-		(pts
 			(xy 181.61 96.52) (xy 179.07 96.52)
 		)
@@
 		(pts
 			(xy 134.62 105.41) (xy 140.97 105.41)
-		)
-		(stroke
-			(width 0)
-			(type default)
-		)
-	)
-	(wire
-		(pts
-			(xy 179.07 100.33) (xy 179.07 101.6)
 		)
 		(stroke
@@
 			)
 		)
-		(property "Footprint" ""
+		(property "Footprint" "Resistor_SMD:R_0508_1220Metric_Pad1.12x2.15mm_HandSolder"
 			(at 157.48 147.828 90)
 			(effects
@@
 	)
 	(symbol
-		(lib_id "Connector_Generic:Conn_01x04")
+		(lib_id "Connector_Generic:Conn_01x02")
 		(at 186.69 96.52 0)
 		(unit 1)
@@
 			)
 		)
-		(property "Footprint" ""
+		(property "Footprint" "Connector_AMASS:AMASS_XT60-F_1x02_P7.20mm_Vertical"
 			(at 186.69 96.52 0)
 			(effects
@@
 			)
 		)
-		(property "Description" "Generic connector, single row, 01x04, script generated (kicad-library-utils/schlib/autogen/connector/)"
+		(property "Description" "Generic connector, single row, 01x02, script generated (kicad-library-utils/schlib/autogen/connector/)"
 			(at 186.69 96.52 0)
 			(effects
@@
 			)
 		)
-		(pin "3"
-		)
 		(pin "2"
 		)
 		(pin "1"
-		)
-		(pin "4"
 		)
 		(instances
@@
 			)
 		)
-		(property "Footprint" ""
+		(property "Footprint" "Resistor_SMD:R_0508_1220Metric_Pad1.12x2.15mm_HandSolder"
 			(at 140.97 144.272 90)
 			(effects
@@
 			)
 		)
-		(property "Footprint" ""
+		(property "Footprint" "Resistor_THT:R_Axial_DIN0309_L9.0mm_D3.2mm_P15.24mm_Horizontal"
 			(at 116.332 118.11 90)
 			(effects
@@
 			)
 		)
-		(property "Footprint" ""
+		(property "Footprint" "Resistor_THT:R_Axial_DIN0309_L9.0mm_D3.2mm_P15.24mm_Horizontal"
 			(at 71.882 102.87 90)
 			(effects
@@
 		)
 		(property "Value" "2k"
-			(at 88.138 114.046 90)
+			(at 87.63 114.3 90)
 			(effects
 				(font
@@
 			)
 		)
-		(property "Footprint" ""
+		(property "Footprint" "Resistor_THT:R_Axial_DIN0309_L9.0mm_D3.2mm_P15.24mm_Horizontal"
 			(at 85.852 113.03 90)
 			(effects
@@
 			)
 		)
-		(property "Footprint" ""
+		(property "Footprint" "Resistor_SMD:R_0508_1220Metric_Pad1.12x2.15mm_HandSolder"
 			(at 166.37 147.828 90)
 			(effects
@@
 			)
 		)
-		(property "Footprint" ""
+		(property "Footprint" "Resistor_SMD:R_0603_1608Metric_Pad0.98x0.95mm_HandSolder"
 			(at 85.852 123.19 90)
 			(effects
@@
 			)
 		)
-		(property "Footprint" ""
+		(property "Footprint" "Resistor_THT:R_Axial_DIN0309_L9.0mm_D3.2mm_P15.24mm_Horizontal"
 			(at 116.332 127 90)
 			(effects
@@
 			)
 		)
-		(property "Footprint" ""
+		(property "Footprint" "Resistor_SMD:R_0508_1220Metric_Pad1.12x2.15mm_HandSolder"
 			(at 149.86 144.272 90)
 			(effects
@@
 			)
 		)
-		(property "Footprint" ""
+		(property "Footprint" "Diode_THT:D_DO-201_P15.24mm_Horizontal"
 			(at 64.77 104.14 0)
 			(effects
@@
 			)
 		)
-		(property "Footprint" ""
+		(property "Footprint" "Resistor_THT:R_Axial_DIN0309_L9.0mm_D3.2mm_P15.24mm_Horizontal"
 			(at 139.192 97.79 90)
 			(effects
@@
 			)
 		)
-		(property "Footprint" ""
+		(property "Footprint" "Capacitor_SMD:C_0805_2012Metric_Pad1.18x1.45mm_HandSolder"
 			(at 171.1452 85.09 0)
 			(effects
@@
 			)
 		)
-		(property "Footprint" ""
+		(property "Footprint" "Capacitor_SMD:C_0805_2012Metric_Pad1.18x1.45mm_HandSolder"
 			(at 171.1452 93.98 0)
 			(effects
@@
 			)
 		)
-		(property "Footprint" ""
+		(property "Footprint" "Diode_THT:D_DO-201_P15.24mm_Horizontal"
 			(at 134.62 97.79 0)
 			(effects

Commit message: finalised product
Parts:
- R31, R37, R38: footprint Resistor_THT:R_Axial_DIN0309_L9.0mm_D3.2mm_P15.24mm_Horizontal -> Resistor_SMD:R_1206_3216Metric
- R39: footprint Resistor_THT:R_Axial_DIN0309_L9.0mm_D3.2mm_P15.24mm_Horizontal -> Resistor_SMD:R_1210_3225Metric_Pad1.30x2.65mm_HandSolder
- R60: footprint Resistor_SMD:R_0603_1608Metric_Pad0.98x0.95mm_HandSolder -> Resistor_SMD:R_1206_3216Metric
Changed lines of the file:
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@@
 			)
 		)
-		(property "Footprint" "Resistor_THT:R_Axial_DIN0309_L9.0mm_D3.2mm_P15.24mm_Horizontal"
+		(property "Footprint" "Resistor_SMD:R_1206_3216Metric"
 			(at 116.332 118.11 90)
 			(effects
@@
 			)
 		)
-		(property "Footprint" "Resistor_THT:R_Axial_DIN0309_L9.0mm_D3.2mm_P15.24mm_Horizontal"
+		(property "Footprint" "Resistor_SMD:R_1206_3216Metric"
 			(at 85.852 113.03 90)
 			(effects
@@
 			)
 		)
-		(property "Footprint" "Resistor_SMD:R_0603_1608Metric_Pad0.98x0.95mm_HandSolder"
+		(property "Footprint" "Resistor_SMD:R_1206_3216Metric"
 			(at 85.852 123.19 90)
 			(effects
@@
 			)
 		)
-		(property "Footprint" "Resistor_THT:R_Axial_DIN0309_L9.0mm_D3.2mm_P15.24mm_Horizontal"
+		(property "Footprint" "Resistor_SMD:R_1206_3216Metric"
 			(at 116.332 127 90)
 			(effects
@@
 			)
 		)
-		(property "Footprint" "Resistor_THT:R_Axial_DIN0309_L9.0mm_D3.2mm_P15.24mm_Horizontal"
+		(property "Footprint" "Resistor_SMD:R_1210_3225Metric_Pad1.30x2.65mm_HandSolder"
 			(at 139.192 97.79 90)
 			(effects

Commit message: near end
Parts:
- R39: footprint Resistor_SMD:R_1210_3225Metric_Pad1.30x2.65mm_HandSolder -> Resistor_THT:R_Axial_DIN0309_L9.0mm_D3.2mm_P15.24mm_Horizontal
Changed lines of the file:
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@@
 			)
 		)
-		(property "Footprint" "Resistor_SMD:R_1210_3225Metric_Pad1.30x2.65mm_HandSolder"
+		(property "Footprint" "Resistor_THT:R_Axial_DIN0309_L9.0mm_D3.2mm_P15.24mm_Horizontal"
 			(at 139.192 97.79 90)
 			(effects

Commit message: bit artık
Parts:
- removed J4: Output, Connector_AMASS:AMASS_XT60-F_1x02_P7.20mm_Vertical, symbol Connector_Generic:Conn_01x02
- added MP3: PACK+, WP-BUTR_7460307:WP-BUTR_7460307, symbol WP-BUTR:WP-BUTR
- added MP4: PACK-, WP-BUTR_7460307:WP-BUTR_7460307, symbol WP-BUTR:WP-BUTR
- added Q8, Q9: HY3610P, Package_TO_SOT_THT:TO-220-3_Vertical, symbol Simulation_SPICE:NMOS
Connections:
- net B_Pos: now also Q9.3 (S); no longer C29.1
- net CD: now also Q8.1 (D), Q9.1 (D)
- net GNDPWR: now also C30.2, MP4.1, MP4.2, MP4.3, MP4.4, MP4.5, MP4.6, MP4.7, MP4.8
- net at D4.2 (A), Q3.3 (S), R34.2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: now also C29.1, MP3.1, MP3.2, MP3.3, MP3.4, MP3.5, MP3.6, MP3.7, MP3.8, Q8.3 (S); no longer C30.2
- net at D4.1 (K), Q3.2 (G), R38.1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: now also Q8.2 (G)
- net at D3.1 (K), Q2.2 (G), R31.1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: now also Q9.2 (G)
Other:
- moved on the sheet: C29, C30

Commit message: BMS DONE IHOPE
Parts:
- removed R31, R37, R60: 2k, Resistor_SMD:R_1206_3216Metric, symbol Device:R
- removed R39: 1M, Resistor_THT:R_Axial_DIN0309_L9.0mm_D3.2mm_P15.24mm_Horizontal, symbol Device:R
- added Q10, Q11: BUK7M27-80EX, Package_TO_SOT_SMD:LFPAK33, symbol Simulation_SPICE:NMOS
- added R25, R31, R37, R39, R60, R73: 47, Resistor_SMD:R_0603_1608Metric_Pad0.98x0.95mm_HandSolder, symbol LibreSolar:R
- D3, D4: footprint Diode_THT:D_DO-201_P15.24mm_Horizontal -> Diode_SMD:D_SMF
- Q2, Q3, Q8, Q9: value HY3610P -> BUK7M27-80EX; footprint Package_TO_SOT_THT:TO-220-3_Vertical -> Package_TO_SOT_SMD:LFPAK33
- R32: footprint Resistor_THT:R_Axial_DIN0309_L9.0mm_D3.2mm_P15.24mm_Horizontal -> Resistor_SMD:R_2512_6332Metric_Pad1.40x3.35mm_HandSolder
- R33, R34, R35, R36: footprint Resistor_SMD:R_0508_1220Metric_Pad1.12x2.15mm_HandSolder -> Resistor_SMD:R_0603_1608Metric_Pad0.98x0.95mm_HandSolder
- R38: value 2k -> 1M; footprint Resistor_SMD:R_1206_3216Metric -> Resistor_SMD:R_2512_6332Metric_Pad1.40x3.35mm_HandSolder
Connections:
- net B_Pos: no longer D3.2 (A), Q2.3 (S), Q9.3 (S), R32.1
- net CD: now also Q2.5 (D), Q3.5 (D), Q8.5 (D), Q9.5 (D), Q10.5 (D), Q11.5 (D); no longer Q2.1 (D), Q3.1 (D), Q8.1 (D), Q9.1 (D)
- net CHG: now also D3.1 (K), R32.2, R25.1, R31.1, R37.1
- net DSG: now also D4.1 (K), R38.2, R39.1, R60.1, R73.1
- net PACK: now also R33.2; no longer R33.1
- net at R34.1: now also R33.1; no longer R33.2
- net PACK+: now reaches C29.1, D4.2 (A), MP3.1, MP3.2, MP3.3, MP3.4, MP3.5, MP3.6, MP3.7, MP3.8, R34.2, R35.1
- net PACK+: now also Q2.1 (S), Q2.2 (S), Q2.3 (S), R38.1, Q10.1 (S), Q10.2 (S), Q10.3 (S), Q11.1 (S), Q11.2 (S), Q11.3 (S); no longer Q3.3 (S), Q8.3 (S)
- net B_POS: now reaches Q3.2 (S), Q8.2 (S)
- net B_POS: now also D3.2 (A), Q3.1 (S), Q3.3 (S), Q8.1 (S), Q8.3 (S), Q9.1 (S), Q9.2 (S), Q9.3 (S), R32.1; no longer D4.1 (K), R38.1
- new net: Q11.4 (G), R73.2
- new net: Q8.4 (G), R25.2
- new net: Q2.4 (G), R39.2
- new net: Q3.4 (G), R31.2
- new net: Q10.4 (G), R60.2
- new net: Q9.4 (G), R37.2
Other:
- moved on the sheet: C29, C30, D3, MP3, MP4, R32, R33, R34, R35, R36
