File: shell-bms.kicad_sch (KiCad schematic)
At the start: 0 parts

Commit message: lots of lots changes. Schematic done NEEDS Review
Connections:
- no-connect marks 0 -> 3
Other:
- added sheet Data_Utils (data_utils.kicad_sch)
- sheet MCU ports: added +3V3, BUZZER, CAN_RX, CAN_TX, FAN1, FAN2, IC_SCL, IC_SDA, PB3, PB4, PB5, STAT_LED, UART_USB_RX, UART_USB_TX; removed none
- sheet Protection ports: added B_Pos; removed none
- sheet ReaderIC ports: added +3V3; removed none
- sheet VIN ports: added +3V3, +5V, Battery_Pozitive; removed none
- company: (none) -> Pehlivan Team
- title: (none) -> Pehli-Shell-BMS

Commit message: son update
Connections:
- no-connect marks 3 -> 4
Other:
- sheet MCU ports: added NTC; removed none
- sheet Protection ports: added none; removed CI_TOP
- sheet ReaderIC ports: added NTC; removed CI_Top
Changed lines of the file:
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@@
+	)
+	(no_connect
+		(at 96.52 64.77)
 	)
 	(no_connect
@@
 	(wire
 		(pts
+			(xy 119.38 87.63) (xy 157.48 87.63)
+		)
+		(stroke
+			(width 0)
+			(type default)
+			(color 255 0 0 1)
+		)
+	)
+	(wire
+		(pts
 			(xy 96.52 115.57) (xy 96.52 127)
 		)
@@
 		(pts
 			(xy 81.28 115.57) (xy 81.28 127)
-		)
-		(stroke
-			(width 0)
-			(type default)
-			(color 0 0 255 1)
-		)
-	)
-	(wire
-		(pts
-			(xy 173.99 113.03) (xy 173.99 104.14)
 		)
 		(stroke
@@
 			)
 		)
+		(pin "NTC" input
+			(at 119.38 87.63 0)
+			(effects
+				(font
+					(size 1.27 1.27)
+				)
+				(justify right)
+			)
+		)
 		(instances
 			(project "shell-bms"
@@
 			)
 		)
-		(pin "CI_TOP" input
-			(at 173.99 113.03 90)
-			(effects
-				(font
-					(size 1.27 1.27)
-				)
-				(justify right)
-			)
-		)
 		(pin "DSG" output
 			(at 166.37 113.03 90)
@@
 			)
 		)
-		(pin "CI_Top" output
-			(at 173.99 104.14 270)
-			(effects
-				(font
-					(size 1.27 1.27)
-				)
-				(justify left)
-			)
-		)
 		(pin "+3V3" input
 			(at 157.48 78.74 180)
 			(effects
 				(font
+					(size 1.27 1.27)
+				)
+				(justify left)
+			)
+		)
+		(pin "NTC" output
+			(at 157.48 87.63 180)
+			(effects
+				(font

Commit message: bit artık
Parts:
- added H1, H2, H3, H4, H5, H6: MountingHole, Mounting_Wuerth:Mounting_Wuerth_WA-SMST-2.25mm_H2.5mm_9774025943, symbol Mechanical:MountingHole

Commit message: BMS DONE IHOPE
Other:
- sheet Data_Utils ports: added PB0, PB1, PB2, PB6, USB+, USB-; removed RXD, TXD
- sheet MCU ports: added PB0, PB1, PB2, PB6, USB+, USB-; removed UART_USB_RX, UART_USB_TX
- sheet Protection ports: added B_POS; removed B_Pos
