File: vin.kicad_sch (KiCad schematic)
At the start: 2 parts

Commit message: lots of lots changes. Schematic done NEEDS Review
Parts:
- added NT1: NetTie_3_Tee, symbol Device:NetTie_3_Tee
- H1: value MountingHole_Pad -> B+
- H2: value MountingHole_Pad -> B-
Connections:
- net at H2.1: now also NT1.3
- net Converter/Voltage_In renamed Battery_Pozitive
- new net GND: NT1.1
- new net GNDPWR: NT1.2
Other:
- note added: "this is f... needed because the f... every component can be fed by amk IC ama MCU takes too much current for amk IC can handle or it burns to ashes"
- company: (none) -> Pehlivan Team
- title: (none) -> VIN

Commit message: son update
Parts:
- H1, H2: footprint (none) -> MountingHole:MountingHole_8.4mm_M8_Pad_Via
- NT1: footprint (none) -> NetTie:NetTie-3_THT_Pad0.3mm
Connections:
- no-connect marks 0 -> 1
Changed lines of the file:
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@@
 		(color 0 0 0 0)
+	)
+	(no_connect
+		(at 140.97 34.29)
 	)
 	(wire
@@
 			)
 		)
-		(property "Footprint" ""
+		(property "Footprint" "NetTie:NetTie-3_THT_Pad0.3mm"
 			(at 86.36 57.15 0)
 			(effects
@@
 			)
 		)
-		(property "Footprint" ""
+		(property "Footprint" "MountingHole:MountingHole_8.4mm_M8_Pad_Via"
 			(at 64.77 49.53 0)
 			(effects
@@
 			)
 		)
-		(property "Footprint" ""
+		(property "Footprint" "MountingHole:MountingHole_8.4mm_M8_Pad_Via"
 			(at 64.77 39.37 0)
 			(effects

Commit message: bit artık
Parts:
- removed H1: B+, MountingHole:MountingHole_8.4mm_M8_Pad_Via, symbol Mechanical:MountingHole_Pad
- removed H2: B-, MountingHole:MountingHole_8.4mm_M8_Pad_Via, symbol Mechanical:MountingHole_Pad
- added MP1: BAT+, WP-BUTR_7460307:WP-BUTR_7460307, symbol WP-BUTR:WP-BUTR
- added MP2: BAT-, WP-BUTR_7460307:WP-BUTR_7460307, symbol WP-BUTR:WP-BUTR
Connections:
- net Battery_Pozitive: now also MP1.1, MP1.2, MP1.3, MP1.4, MP1.5, MP1.6, MP1.7, MP1.8
- net at NT1.3: now also MP2.1, MP2.2, MP2.3, MP2.4, MP2.5, MP2.6, MP2.7, MP2.8

Commit message: BMS DONE IHOPE
Parts:
- removed NT1: NetTie_3_Tee, NetTie:NetTie-3_THT_Pad0.3mm, symbol Device:NetTie_3_Tee
- added NT1, NT2, NT3: NetTie_2, NetTie:NetTie-2_THT_Pad0.3mm, symbol Device:NetTie_2
Connections:
- net GND: now also NT1.2, NT2.2, NT3.2
- net GNDPWR: now also MP2.1, MP2.2, MP2.3, MP2.4, MP2.5, MP2.6, MP2.7, MP2.8, NT1.1, NT2.1, NT3.1
